Commit message: clear

File: assets/doosan/doosan_origin.urdf (robot description, URDF)
Before this commit: robot Doosan_loz, 8 links, 7 joints
Links:
- link Base_0: geometry collision mesh filename=m0609_collision/MF0609_0_0.dae scale=0.001 0.001 0.001; visual mesh filename=m0609_collision/MF0609_0_0.dae scale=0.001 0.001 0.001
- link link1: geometry collision mesh filename=m0609_collision/MF0609_1_0.dae scale=0.001 0.001 0.001; visual mesh filename=m0609_collision/MF0609_1_0.dae scale=0.001 0.001 0.001
- link link2: geometry collision mesh filename=m0609_collision/MF0609_2_0.dae scale=0.001 0.001 0.001; collision mesh filename=m0609_collision/MF0609_2_1.dae scale=0.001 0.001 0.001
- link link3: geometry collision mesh filename=m0609_collision/MF0609_3_0.dae scale=0.001 0.001 0.001; visual mesh filename=m0609_collision/MF0609_3_0.dae scale=0.001 0.001 0.001
- link link4: geometry collision mesh filename=m0609_collision/MF0609_4_0.dae scale=0.001 0.001 0.001; collision mesh filename=m0609_collision/MF0609_4_1.dae scale=0.001 0.001 0.001
- link link5: geometry collision mesh filename=m0609_collision/MF0609_5_0.dae scale=0.001 0.001 0.001; visual mesh filename=m0609_collision/MF0609_5_0.dae scale=0.001 0.001 0.001
- link link6: geometry collision mesh filename=m0609_collision/MF0609_6_0.dae scale=0.001 0.001 0.001; visual mesh filename=m0609_collision/MF0609_6_0.dae scale=0.001 0.001 0.001

File: assets/doosan/plane.urdf (robot description, URDF)
Before this commit: robot plane, 1 links, 0 joints
Links:
- link planeLink: geometry collision box size=30 30 10; visual mesh filename=assets/doosan/obj_plane/plane_transparent.obj scale=1 1 1

File: assets/tote/tote_bin.urdf (robot description, URDF)
Before this commit: robot toteA_large, 1 links, 0 joints
Links:
- link base_link: geometry collision mesh filename=assets/doosan/m0609_collision/Bin.STL scale=0.1 0.1 0.1; visual mesh filename=assets/doosan/m0609_collision/Bin.STL scale=0.1 0.1 0.1
