Commit message: enable_base_and_framework

File: assets/doosan/Cabin.urdf (robot description, URDF)
Before this commit: robot m0609, 1 links, 0 joints
Links:
- link Cabin: geometry visual mesh filename=assets/doosan/m0609_collision/Cabin_khung.STL scale=0.01 0.01 0.01

File: assets/doosan/base_doosan.urdf (robot description, URDF)
Before this commit: robot m0609, 1 links, 0 joints
Links:
- link base_0: geometry visual mesh filename=assets/doosan/m0609_collision/base_doosan.STL scale=0.01 0.01 0.01
